Commit message: ar_dual: shared upper-body model, AmazingHand mesh, flip4, left-arm zero offsets
- humanoi_upper.xacro: torso/pole/head/camera + both arms + hands, shared
  by the real dual-arm system and the Gazebo full robot; arm_control.xacro
  picks real/mock/gz hardware
- AmazingHand mesh (Pollen AH_Right, Apache-2.0) flattened by
  mjcf_flatten.py; collision rules for the hands in the SRDF
- ar_arm.xacro: flip4 (right arm J4 zero 180 deg off) and off1..off6:
  measured joint zero offsets, applied as a fixed rotation link_N_raw ->
  link_N about the joint axis. Firmware angles and taught poses unchanged.
- left arm offsets -7 -2 0 -7 +19 +15 deg (each joint levelled with a
  spirit level, program value read; offset = -reading), checked in RViz

Co-Authored-By: Claude Opus 5.5 <noreply@anthropic.com>

File: ar4_ws/src/ar_dual/urdf/ar_arm.xacro (robot description, xacro)
@@ -3,7 +3,24 @@
      เพื่อใส่แขน AR4 สองตัวในโมเดลเดียว (left_ / right_) — สร้างด้วยสคริปต์แทนที่ชื่อเท่านั้น
      ค่าเรขาคณิต/ลิมิต/mesh เหมือนต้นฉบับทุกตัว (mesh ยังอ่านจากแพ็กเกจ ar_description)
-     เพิ่ม dir1..dir6 (ค่าเริ่ม 1): -1 = กลับทิศหมุนของข้อนั้นในโมเดล ให้ตรงกับแขนที่ประกอบข้อนั้นกลับด้าน -->
+     เพิ่ม dir1..dir6 (ค่าเริ่ม 1): -1 = กลับทิศหมุนของข้อนั้นในโมเดล ให้ตรงกับแขนที่ประกอบข้อนั้นกลับด้าน
+     เพิ่ม flip4 (ค่าเริ่ม 0): 1 = ศูนย์ของข้อ 4 อยู่ห่างจากต้นฉบับ 180° (ข้อมือทั้งชุดหมุนครึ่งรอบ — ชุดข้อ 5 อยู่อีกฝั่ง
+     และข้อ 5 ดูงอกลับทิศ) ค่ามุมจากเฟิร์มแวร์ไม่เปลี่ยน แค่หมุนเฟรมลูกของข้อ 4 รอบแกนตัวเอง 180°
+     เพิ่ม off1..off6 (องศา ค่าเริ่ม 0): มุมจริงของข้อ − มุมที่เฟิร์มแวร์นับ (วัดจากแขนจริง) — เฟรม link_N หมุนต่อจาก
+     link_N_raw (ตามมุมที่นับได้) รอบแกนเดียวกันอีก offN · มุมที่โปรแกรมเห็น/สั่ง และท่าที่สอนไว้ไม่เปลี่ยน แค่โมเดลตรงของจริง
+     ต่างจากต้นฉบับ: effort = 100 ทุกข้อ และ joint_2 velocity = 0.5 (ต้นฉบับตั้ง effort 0 / velocity 0 —
+     แขนจริงไม่ได้อ่านค่านี้ แต่ใน Gazebo effort 0 = มอเตอร์ไม่มีแรง แขนห้อยตกจนชน hard-stop) -->
 <robot xmlns:xacro="http://wiki.ros.org/xacro">
-  <xacro:macro name="ar_arm" params="prefix parent *origin dir1:=1 dir2:=1 dir3:=1 dir4:=1 dir5:=1 dir6:=1">
+  <!-- ศูนย์ข้อต่อจริงห่างจากที่เฟิร์มแวร์นับ: ข้อ revolute หมุน link_N_raw ตามมุมที่นับ แล้วหมุนต่ออีก offset รอบแกนเดียวกัน
+       (rpy = แกนข้อ × offset) — link_N คือเฟรมจริงของชิ้นแขน mesh/มือ/กล้องอ้างเฟรมนี้เหมือนเดิม -->
+  <xacro:macro name="zero_offset" params="prefix n rpy">
+    <link name="${prefix}link_${n}_raw"/>
+    <joint name="${prefix}joint_${n}_zero" type="fixed">
+      <parent link="${prefix}link_${n}_raw"/>
+      <child link="${prefix}link_${n}"/>
+      <origin rpy="${rpy}" xyz="0 0 0"/>
+    </joint>
+  </xacro:macro>
+  <xacro:macro name="ar_arm" params="prefix parent *origin dir1:=1 dir2:=1 dir3:=1 dir4:=1 dir5:=1 dir6:=1 flip4:=0
+                                   off1:=0 off2:=0 off3:=0 off4:=0 off5:=0 off6:=0">
     <joint name="${prefix}base_joint" type="fixed">
       <xacro:insert_block name="origin" />
@@ -58,8 +75,9 @@
       <origin rpy="${pi} 0 0" xyz="0 0 0.003445"/>
       <parent link="${prefix}base_link"/>
-      <child link="${prefix}link_1"/>
+      <child link="${prefix}link_1_raw"/>
       <axis xyz="${float(dir1) * 0} ${float(dir1) * 0} ${float(dir1) * 1}"/>
-      <limit lower="${-170.0 / 180.0 * pi}" upper="${170.0 / 180.0 * pi}" effort="0" velocity="0.5"/>
-    </joint>
+      <limit lower="${-170.0 / 180.0 * pi}" upper="${170.0 / 180.0 * pi}" effort="100" velocity="0.5"/>
+    </joint>
+    <xacro:zero_offset prefix="${prefix}" n="1" rpy="0 0 ${float(off1) * pi / 180.0 * float(dir1)}"/>
     <link name="${prefix}link_2">
       <inertial>
@@ -87,8 +105,9 @@
       <origin rpy="1.5708 0.5236 -1.5708" xyz="0 0.064146 -0.16608"/>
       <parent link="${prefix}link_1"/>
-      <child link="${prefix}link_2"/>
+      <child link="${prefix}link_2_raw"/>
       <axis xyz="${float(dir2) * 0} ${float(dir2) * 0} ${float(dir2) * -1}"/>
-      <limit lower="${-42.0 / 180.0 * pi}" upper="${90.0 / 180.0 * pi}" effort="0.5" velocity="0"/>
-    </joint>
+      <limit lower="${-42.0 / 180.0 * pi}" upper="${90.0 / 180.0 * pi}" effort="100" velocity="0.5"/>
+    </joint>
+    <xacro:zero_offset prefix="${prefix}" n="2" rpy="0 0 ${-float(off2) * pi / 180.0 * float(dir2)}"/>
     <link name="${prefix}link_3">
       <inertial>
@@ -116,8 +135,9 @@
       <origin rpy="0 0 -2.61799" xyz="0.1525 -0.26414 0"/>
       <parent link="${prefix}link_2"/>
-      <child link="${prefix}link_3"/>
+      <child link="${prefix}link_3_raw"/>
       <axis xyz="${float(dir3) * 0} ${float(dir3) * 0} ${float(dir3) * -1}"/>
-      <limit lower="${-89.0 / 180.0 * pi}" upper="${52.0 / 180.0 * pi}" effort="0" velocity="0.5"/>
-    </joint>
+      <limit lower="${-89.0 / 180.0 * pi}" upper="${52.0 / 180.0 * pi}" effort="100" velocity="0.5"/>
+    </joint>
+    <xacro:zero_offset prefix="${prefix}" n="3" rpy="0 0 ${-float(off3) * pi / 180.0 * float(dir3)}"/>
     <link name="${prefix}link_4">
       <inertial>
@@ -143,10 +163,12 @@
     </link>
     <joint name="${prefix}joint_4" type="revolute">
-      <origin rpy="1.5708 -1.2554 -1.5708" xyz="0 0 0.00675"/>
+      <!-- flip4: ต้นฉบับ × หมุนรอบแกนข้อ 4 (z) 180° — คำนวณไว้แล้ว (ตรวจย้อนกลับ ผิดพลาด < 1e-15) -->
+      <origin rpy="${'-1.5708 1.2554 1.570793' if int(flip4) else '1.5708 -1.2554 -1.5708'}" xyz="0 0 0.00675"/>
       <parent link="${prefix}link_3"/>
-      <child link="${prefix}link_4"/>
+      <child link="${prefix}link_4_raw"/>
       <axis xyz="${float(dir4) * 0} ${float(dir4) * 0} ${float(dir4) * -1}"/>
-      <limit lower="${-165.0 / 180.0 * pi}" upper="${165.0 / 180.0 * pi}" effort="0" velocity="0.5"/>
-    </joint>
+      <limit lower="${-165.0 / 180.0 * pi}" upper="${165.0 / 180.0 * pi}" effort="100" velocity="0.5"/>
+    </joint>
+    <xacro:zero_offset prefix="${prefix}" n="4" rpy="0 0 ${-float(off4) * pi / 180.0 * float(dir4)}"/>
     <link name="${prefix}link_5">
       <inertial>
@@ -174,8 +196,9 @@
       <origin rpy="${pi} 0 -2.8262" xyz="0 0 -0.22225"/>
       <parent link="${prefix}link_4"/>
-      <child link="${prefix}link_5"/>
+      <child link="${prefix}link_5_raw"/>
       <axis xyz="${float(dir5) * 1} ${float(dir5) * 0} ${float(dir5) * 0}"/>
-      <limit lower="${-105.0 / 180.0 * pi}" upper="${105.0 / 180.0 * pi}" effort="0" velocity="0.5"/>
-    </joint>
+      <limit lower="${-105.0 / 180.0 * pi}" upper="${105.0 / 180.0 * pi}" effort="100" velocity="0.5"/>
+    </joint>
+    <xacro:zero_offset prefix="${prefix}" n="5" rpy="${float(off5) * pi / 180.0 * float(dir5)} 0 0"/>
     <link name="${prefix}link_6">
       <inertial>
@@ -203,8 +226,9 @@
       <origin rpy="0 0 3.1416" xyz="-0.000294 0 0.02117"/>
       <parent link="${prefix}link_5"/>
-      <child link="${prefix}link_6"/>
+      <child link="${prefix}link_6_raw"/>
       <axis xyz="${float(dir6) * 0} ${float(dir6) * 0} ${float(dir6) * 1}"/>
-      <limit lower="${-155.0 / 180.0 * pi}" upper="${155.0 / 180.0 * pi}" effort="0" velocity="0.5"/>
-    </joint>
+      <limit lower="${-155.0 / 180.0 * pi}" upper="${155.0 / 180.0 * pi}" effort="100" velocity="0.5"/>
+    </joint>
+    <xacro:zero_offset prefix="${prefix}" n="6" rpy="0 0 ${float(off6) * pi / 180.0 * float(dir6)}"/>
   </xacro:macro>
 </robot>

File: ar4_ws/src/ar_dual/urdf/humanoi_arms.urdf.xacro (robot description, xacro)
@@ -1,10 +1,5 @@
 <?xml version="1.0"?>
-<!-- Humanoi: แขน AR4 สองตัว (ซ้าย/ขวา) ติดสองข้างเสากลาง + เสา หัว กล้อง (ไว้ให้ MoveIt เช็กการชน)
-  เฟรมราก "torso" = กึ่งกลางระหว่างฐานแขนสองตัว ที่ความสูงหัวไหล่: X ไปหน้าหุ่น, Y ไปซ้ายหุ่น, Z ขึ้น
-  ฐานแขน (base_link ของ AR4: Z = แกน J1 ชี้ออกจากผิวที่ยึด) ยึดกับเสาแนวนอน ห่างกัน 11 cm (วัดจริง)
-  - ซ้าย: Z ชี้ไปซ้ายหุ่น, X ไปหน้า, Y ลง — ได้จาก hand-eye calibration วันที่ 15 ต.ค. (ทิศขึ้น = -Y ของฐาน)
-  - ขวา: กลับด้านจากซ้าย (กล่องมอเตอร์ J1 ห้อยลงเหมือนกันตามรูป) — Z ชี้ไปขวา, X ไปหลัง, Y ลง
-    ** เดาจากรูป ยังไม่ได้วัด — ถ้าโมเดลแขนขวาใน RViz ไม่ตรงกับแขนจริงให้แก้ right_rpy **
-  เสา/หัว/กล้อง = กล่องและทรงกลมคร่าวๆ (เผื่อใหญ่ไว้) ใช้แค่กันชนใน MoveIt
+<!-- Humanoi: แขน AR4 สองตัว (ซ้าย/ขวา) ติดสองข้างเสากลาง + เสา หัว กล้อง มือ — สำหรับระบบแขนจริง (ไม่มีฐานล้อ)
+  เรขาคณิตทั้งหมดอยู่ใน humanoi_upper.xacro (ใช้ร่วมกับหุ่นเต็มตัวใน Gazebo) — แก้ขนาดที่นั่น
   ฮาร์ดแวร์แต่ละแขน: left_hw / right_hw = real (Teensy ผ่านไดรเวอร์ของผู้ขาย) หรือ mock (จำลอง ไม่ต่อบอร์ด)
   calibrate ไม่ทำใน ROS (ไดรเวอร์ผู้ขายบล็อก ~2 นาที/แขน และ USB มักหลุดระหว่างนั้น) — ใช้ scripts/ar_calibrate.py
@@ -15,82 +10,7 @@
   <xacro:arg name="left_hw" default="real"/>
   <xacro:arg name="right_hw" default="real"/>
-  <xacro:property name="half_gap" value="0.055"/>
-  <xacro:property name="left_rpy" value="${-pi/2} 0 0"/>
-  <xacro:property name="right_rpy" value="${-pi/2} 0 ${pi}"/>
-  <xacro:include filename="$(find ar_dual)/urdf/ar_arm.xacro"/>
-  <link name="torso">
-    <!-- เสาอะลูมิเนียมโปรไฟล์ (หน้ากว้าง ~8 cm ตามรูป) ยาวลงไปถึงฐานล้อ -->
-    <collision>
-      <origin xyz="0.01 0 -0.60" rpy="0 0 0"/>
-      <geometry><box size="0.10 0.08 1.40"/></geometry>
-    </collision>
-    <!-- หัว (หมวกกันน็อก) เหนือหัวไหล่ -->
-    <collision>
-      <origin xyz="0.02 0 0.27" rpy="0 0 0"/>
-      <geometry><sphere radius="0.16"/></geometry>
-    </collision>
-    <!-- กล้อง Astra Pro หน้าเสาใต้หัวไหล่ (ตำแหน่งจาก hand-eye) -->
-    <collision>
-      <origin xyz="0.095 0.009 -0.048" rpy="0 0 0"/>
-      <geometry><box size="0.05 0.17 0.05"/></geometry>
-    </collision>
-    <visual>
-      <origin xyz="0.01 0 -0.60" rpy="0 0 0"/>
-      <geometry><box size="0.10 0.08 1.40"/></geometry>
-      <material name="pole"><color rgba="0.75 0.75 0.78 1"/></material>
-    </visual>
-    <visual>
-      <origin xyz="0.02 0 0.27" rpy="0 0 0"/>
-      <geometry><sphere radius="0.16"/></geometry>
-      <material name="head"><color rgba="0.1 0.1 0.1 1"/></material>
-    </visual>
-    <visual>
-      <origin xyz="0.095 0.009 -0.048" rpy="0 0 0"/>
-      <geometry><box size="0.05 0.17 0.05"/></geometry>
-      <material name="camera"><color rgba="0.2 0.2 0.25 1"/></material>
-    </visual>
-  </link>
-  <xacro:ar_arm prefix="left_" parent="torso">
-    <origin xyz="0 ${half_gap} 0" rpy="${left_rpy}"/>
-  </xacro:ar_arm>
-  <!-- แขนขวา: J5 หมุนกลับทิศกับแขนซ้าย (ผู้ใช้ยืนยันจากของจริง 16 ต.ค. — ข้อมือประกอบกลับด้าน)
-       เฟิร์มแวร์ยังรายงานมุมแบบเดิม จึงกลับทิศแกนในโมเดลแทน ให้ RViz/MoveIt ตรงกับแขนจริง
-       ถ้าเจอข้ออื่นกลับทิศอีก ใส่ dirN="-1" เพิ่มตรงนี้ -->
-  <xacro:ar_arm prefix="right_" parent="torso" dir5="-1">
-    <origin xyz="0 ${-half_gap} 0" rpy="${right_rpy}"/>
-  </xacro:ar_arm>
-  <!-- ros2_control ของแต่ละแขน: ลิมิตเป็นตัวเลขจริง (ไฟล์ของผู้ขายเขียน {..} ไม่มี $ จึง parse ไม่ผ่าน) -->
-  <xacro:macro name="arm_joint" params="name lo hi init">
-    <joint name="${name}">
-      <command_interface name="position">
-        <param name="min">${lo * pi / 180}</param>
-        <param name="max">${hi * pi / 180}</param>
-      </command_interface>
-      <state_interface name="position">
-        <param name="initial_value">${init}</param>
-      </state_interface>
-    </joint>
-  </xacro:macro>
-  <xacro:macro name="arm_control" params="prefix hw port">
-    <ros2_control name="${prefix}arm" type="system">
-      <hardware>
-        <xacro:if value="${hw == 'real'}">
-          <plugin>ar_hardware_interface/ARHardwareInterface</plugin>
-          <param name="serial_port">${port}</param>
-          <param name="calibrate">False</param>
-        </xacro:if>
-        <xacro:unless value="${hw == 'real'}">
-          <plugin>mock_components/GenericSystem</plugin>
-        </xacro:unless>
-      </hardware>
-      <!-- initial_value = ท่าพักหลัง calibrate (ใช้ตอน mock) -->
-      <xacro:arm_joint name="${prefix}joint_1" lo="-170" hi="170" init="0.0"/>
-      <xacro:arm_joint name="${prefix}joint_2" lo="-42" hi="90" init="-0.1019"/>
-      <xacro:arm_joint name="${prefix}joint_3" lo="-89" hi="52" init="0.0"/>
-      <xacro:arm_joint name="${prefix}joint_4" lo="-165" hi="165" init="0.0"/>
-      <xacro:arm_joint name="${prefix}joint_5" lo="-105" hi="105" init="-0.9103"/>
-      <xacro:arm_joint name="${prefix}joint_6" lo="-155" hi="155" init="0.0"/>
-    </ros2_control>
-  </xacro:macro>
+  <xacro:include filename="$(find ar_dual)/urdf/humanoi_upper.xacro"/>
+  <xacro:include filename="$(find ar_dual)/urdf/arm_control.xacro"/>
+  <xacro:humanoi_upper/>
   <xacro:arm_control prefix="left_" hw="$(arg left_hw)" port="$(arg left_port)"/>
   <xacro:arm_control prefix="right_" hw="$(arg right_hw)" port="$(arg right_port)"/>
