Commit message: Joint zero trims in the Teensy: program numbers = real angles
Each left-arm joint was levelled with a spirit level and the program
value read; the trims are minus those readings (-7 -2 0 -7 +19 +15 deg).

- firmware AR4_ROS2_seq v3: JZ / JZ=a,b,c,d,e,f stored in EEPROM;
  reported angle = counted + trim, MT subtracts it. Calibration, rest
  and real travel unchanged. JV answers JVseq3.
- ar_dual/config/zero_trims.yaml is the single source: joint limits in
  ar_arm.xacro / arm_control.xacro and ar_program limits(arm) shift by
  the trims; after_calibrate pose (left J1 J2 J4 J5 J6 -> 0) used by
  ar_calibrate.py --arm, the MoveIt rest state and the sim start pose
- ar_zero.py: check / --apply the board trims against the yaml
- model-only offsets of the left arm back to 0 (board does it now)
- left arm hand model is now the left-hand kit (thumb was on the wrong
  side), right arm gets the right-hand mesh
- check_pose / _round_in take the arm for its limits

Co-Authored-By: Claude Opus 5.5 <noreply@anthropic.com>

File: ar4_ws/src/ar_dual/urdf/ar_arm.xacro (robot description, xacro)
@@ -8,4 +8,5 @@
      เพิ่ม off1..off6 (องศา ค่าเริ่ม 0): มุมจริงของข้อ − มุมที่เฟิร์มแวร์นับ (วัดจากแขนจริง) — เฟรม link_N หมุนต่อจาก
      link_N_raw (ตามมุมที่นับได้) รอบแกนเดียวกันอีก offN · มุมที่โปรแกรมเห็น/สั่ง และท่าที่สอนไว้ไม่เปลี่ยน แค่โมเดลตรงของจริง
+     ลิมิตข้อต่อเลื่อนตามค่าชดเชยศูนย์ในบอร์ด (config/zero_trims.yaml) — ตัวเลขเปลี่ยน ช่วงหมุนจริงเท่าเดิม
      ต่างจากต้นฉบับ: effort = 100 ทุกข้อ และ joint_2 velocity = 0.5 (ต้นฉบับตั้ง effort 0 / velocity 0 —
      แขนจริงไม่ได้อ่านค่านี้ แต่ใน Gazebo effort 0 = มอเตอร์ไม่มีแรง แขนห้อยตกจนชน hard-stop) -->
@@ -13,4 +14,5 @@
   <!-- ศูนย์ข้อต่อจริงห่างจากที่เฟิร์มแวร์นับ: ข้อ revolute หมุน link_N_raw ตามมุมที่นับ แล้วหมุนต่ออีก offset รอบแกนเดียวกัน
        (rpy = แกนข้อ × offset) — link_N คือเฟรมจริงของชิ้นแขน mesh/มือ/กล้องอ้างเฟรมนี้เหมือนเดิม -->
+  <xacro:property name="ar_zero_trims" value="${xacro.load_yaml('$(find ar_dual)/config/zero_trims.yaml')}"/>
   <xacro:macro name="zero_offset" params="prefix n rpy">
     <link name="${prefix}link_${n}_raw"/>
@@ -23,4 +25,6 @@
   <xacro:macro name="ar_arm" params="prefix parent *origin dir1:=1 dir2:=1 dir3:=1 dir4:=1 dir5:=1 dir6:=1 flip4:=0
                                    off1:=0 off2:=0 off3:=0 off4:=0 off5:=0 off6:=0">
+    <!-- ค่าชดเชยศูนย์ในบอร์ดของแขนนี้ (config/zero_trims.yaml ตามชื่อ prefix) — ตัวเลขข้อต่อเลื่อนไป ลิมิตเลื่อนตาม -->
+    <xacro:property name="zt" value="${[float(v) for v in ar_zero_trims.get(prefix[:-1], [0] * 6)]}"/>
     <joint name="${prefix}base_joint" type="fixed">
       <xacro:insert_block name="origin" />
@@ -77,5 +81,5 @@
       <child link="${prefix}link_1_raw"/>
       <axis xyz="${float(dir1) * 0} ${float(dir1) * 0} ${float(dir1) * 1}"/>
-      <limit lower="${-170.0 / 180.0 * pi}" upper="${170.0 / 180.0 * pi}" effort="100" velocity="0.5"/>
+      <limit lower="${(-170.0 + zt[0]) / 180.0 * pi}" upper="${(170.0 + zt[0]) / 180.0 * pi}" effort="100" velocity="0.5"/>
     </joint>
     <xacro:zero_offset prefix="${prefix}" n="1" rpy="0 0 ${float(off1) * pi / 180.0 * float(dir1)}"/>
@@ -107,5 +111,5 @@
       <child link="${prefix}link_2_raw"/>
       <axis xyz="${float(dir2) * 0} ${float(dir2) * 0} ${float(dir2) * -1}"/>
-      <limit lower="${-42.0 / 180.0 * pi}" upper="${90.0 / 180.0 * pi}" effort="100" velocity="0.5"/>
+      <limit lower="${(-42.0 + zt[1]) / 180.0 * pi}" upper="${(90.0 + zt[1]) / 180.0 * pi}" effort="100" velocity="0.5"/>
     </joint>
     <xacro:zero_offset prefix="${prefix}" n="2" rpy="0 0 ${-float(off2) * pi / 180.0 * float(dir2)}"/>
@@ -137,5 +141,5 @@
       <child link="${prefix}link_3_raw"/>
       <axis xyz="${float(dir3) * 0} ${float(dir3) * 0} ${float(dir3) * -1}"/>
-      <limit lower="${-89.0 / 180.0 * pi}" upper="${52.0 / 180.0 * pi}" effort="100" velocity="0.5"/>
+      <limit lower="${(-89.0 + zt[2]) / 180.0 * pi}" upper="${(52.0 + zt[2]) / 180.0 * pi}" effort="100" velocity="0.5"/>
     </joint>
     <xacro:zero_offset prefix="${prefix}" n="3" rpy="0 0 ${-float(off3) * pi / 180.0 * float(dir3)}"/>
@@ -168,5 +172,5 @@
       <child link="${prefix}link_4_raw"/>
       <axis xyz="${float(dir4) * 0} ${float(dir4) * 0} ${float(dir4) * -1}"/>
-      <limit lower="${-165.0 / 180.0 * pi}" upper="${165.0 / 180.0 * pi}" effort="100" velocity="0.5"/>
+      <limit lower="${(-165.0 + zt[3]) / 180.0 * pi}" upper="${(165.0 + zt[3]) / 180.0 * pi}" effort="100" velocity="0.5"/>
     </joint>
     <xacro:zero_offset prefix="${prefix}" n="4" rpy="0 0 ${-float(off4) * pi / 180.0 * float(dir4)}"/>
@@ -198,5 +202,5 @@
       <child link="${prefix}link_5_raw"/>
       <axis xyz="${float(dir5) * 1} ${float(dir5) * 0} ${float(dir5) * 0}"/>
-      <limit lower="${-105.0 / 180.0 * pi}" upper="${105.0 / 180.0 * pi}" effort="100" velocity="0.5"/>
+      <limit lower="${(-105.0 + zt[4]) / 180.0 * pi}" upper="${(105.0 + zt[4]) / 180.0 * pi}" effort="100" velocity="0.5"/>
     </joint>
     <xacro:zero_offset prefix="${prefix}" n="5" rpy="${float(off5) * pi / 180.0 * float(dir5)} 0 0"/>
@@ -228,5 +232,5 @@
       <child link="${prefix}link_6_raw"/>
       <axis xyz="${float(dir6) * 0} ${float(dir6) * 0} ${float(dir6) * 1}"/>
-      <limit lower="${-155.0 / 180.0 * pi}" upper="${155.0 / 180.0 * pi}" effort="100" velocity="0.5"/>
+      <limit lower="${(-155.0 + zt[5]) / 180.0 * pi}" upper="${(155.0 + zt[5]) / 180.0 * pi}" effort="100" velocity="0.5"/>
     </joint>
     <xacro:zero_offset prefix="${prefix}" n="6" rpy="0 0 ${float(off6) * pi / 180.0 * float(dir6)}"/>

File: ar4_ws/src/ar_dual/urdf/arm_control.xacro (robot description, xacro)
@@ -4,4 +4,5 @@
   ลิมิตเป็นตัวเลขจริง (ไฟล์ของผู้ขายเขียน {..} ไม่มี $ จึง parse ไม่ผ่าน)
   initial_value = ท่าพักหลัง calibrate (ใช้ตอน mock / ซิม)
+  ลิมิต / ท่าพัก = ค่าของผู้ขาย + ค่าชดเชยศูนย์ในบอร์ด (config/zero_trims.yaml) ของแขนนั้น
 -->
 <robot xmlns:xacro="http://wiki.ros.org/xacro">
@@ -18,4 +19,9 @@
   </xacro:macro>
   <xacro:macro name="arm_control" params="prefix hw port:=none">
+    <!-- ค่าชดเชยศูนย์ในบอร์ดของแขนนี้ (ar_dual/config/zero_trims.yaml) — ลิมิตและท่าพักเลื่อนตาม -->
+    <xacro:property name="zcfg" value="${xacro.load_yaml('$(find ar_dual)/config/zero_trims.yaml')}"/>
+    <xacro:property name="zt" value="${[float(v) for v in zcfg.get(prefix[:-1], [0] * 6)]}"/>
+    <!-- ท่าหลัง calibrate (after_calibrate มุมจริง องศา) แทนท่าพักของเฟิร์มแวร์ ในข้อที่กำหนด -->
+    <xacro:property name="ac" value="${dict((int(k), float(v)) for k, v in ((zcfg.get('after_calibrate') or dict()).get(prefix[:-1]) or dict()).items())}"/>
     <ros2_control name="${prefix}arm" type="system">
       <hardware>
@@ -34,10 +40,10 @@
         </xacro:if>
       </hardware>
-      <xacro:arm_joint name="${prefix}joint_1" lo="-170" hi="170" init="0.0"/>
-      <xacro:arm_joint name="${prefix}joint_2" lo="-42" hi="90" init="-0.1019"/>
-      <xacro:arm_joint name="${prefix}joint_3" lo="-89" hi="52" init="0.0"/>
-      <xacro:arm_joint name="${prefix}joint_4" lo="-165" hi="165" init="0.0"/>
-      <xacro:arm_joint name="${prefix}joint_5" lo="-105" hi="105" init="-0.9103"/>
-      <xacro:arm_joint name="${prefix}joint_6" lo="-155" hi="155" init="0.0"/>
+      <xacro:arm_joint name="${prefix}joint_1" lo="${-170 + zt[0]}" hi="${170 + zt[0]}" init="${ac[1] * pi / 180 if 1 in ac else 0.0 + zt[0] * pi / 180}"/>
+      <xacro:arm_joint name="${prefix}joint_2" lo="${-42 + zt[1]}" hi="${90 + zt[1]}" init="${ac[2] * pi / 180 if 2 in ac else -0.1019 + zt[1] * pi / 180}"/>
+      <xacro:arm_joint name="${prefix}joint_3" lo="${-89 + zt[2]}" hi="${52 + zt[2]}" init="${ac[3] * pi / 180 if 3 in ac else 0.0 + zt[2] * pi / 180}"/>
+      <xacro:arm_joint name="${prefix}joint_4" lo="${-165 + zt[3]}" hi="${165 + zt[3]}" init="${ac[4] * pi / 180 if 4 in ac else 0.0 + zt[3] * pi / 180}"/>
+      <xacro:arm_joint name="${prefix}joint_5" lo="${-105 + zt[4]}" hi="${105 + zt[4]}" init="${ac[5] * pi / 180 if 5 in ac else -0.9103 + zt[4] * pi / 180}"/>
+      <xacro:arm_joint name="${prefix}joint_6" lo="${-155 + zt[5]}" hi="${155 + zt[5]}" init="${ac[6] * pi / 180 if 6 in ac else 0.0 + zt[5] * pi / 180}"/>
     </ros2_control>
   </xacro:macro>

File: ar4_ws/src/ar_dual/urdf/humanoi_upper.xacro (robot description, xacro)
@@ -70,6 +70,8 @@
     <!-- แขนซ้าย: ศูนย์ข้อต่อจริง (off องศา = มุมจริง − มุมที่โปรแกรมบอก) — 26 ต.ค. ผู้ใช้จัดแต่ละข้อให้ตรงด้วยระดับน้ำ
          (มุมจริง 0) แล้วอ่านค่าในโปรแกรม: ข้อ 1 7 · ข้อ 2 2 · ข้อ 3 0 · ข้อ 4 7 · ข้อ 5 −19 · ข้อ 6 −15 -> off = −ค่าที่อ่าน
-         (ข้อไหนในโมเดลเบี้ยวกว่าเดิม = กลับเครื่องหมายข้อนั้น) -->
-    <xacro:ar_arm prefix="left_" parent="torso" off1="-7" off2="-2" off3="0" off4="-7" off5="19" off6="15">
+         (ข้อไหนในโมเดลเบี้ยวกว่าเดิม = กลับเครื่องหมายข้อนั้น)
+         ทุกข้อย้ายไปชดเชยในบอร์ดแล้ว (config/zero_trims.yaml -> ตัวเลขในโปรแกรม = มุมจริง) off จึงเป็น 0 ทุกข้อ
+         ข้อที่ย้ายไปบอร์ด: off ข้อนั้น = 0 (ไม่งั้นชดเชยซ้ำสองที่) — off ใช้กับข้อที่ยังไม่ได้ย้ายเท่านั้น -->
+    <xacro:ar_arm prefix="left_" parent="torso" off1="0" off2="0" off3="0" off4="0" off5="0" off6="0">
       <origin xyz="0 ${up_half_gap} 0" rpy="${up_left_rpy}"/>
     </xacro:ar_arm>
@@ -85,11 +87,13 @@
     <xacro:if value="${left_hand}">
       <!-- เทียบรูปจริงท่าพักหลัง calibrate (21 ต.ค.): ฝ่ามือหันเข้าเสา/ขึ้นบน = หมุน 90° จากโมเดล
-           ตัวยึดกลมสีขาวระหว่างหน้าแปลนกับมือ ~25 มม. (ประเมินจากรูป — วัดจริงแล้วแก้ mount_offset) -->
-      <xacro:amazinghand prefix="left_" parent="left_link_6" mount_offset="0.025" mount_yaw="${pi/2}"/>
+           ตัวยึดกลมสีขาวระหว่างหน้าแปลนกับมือ ~25 มม. (ประเมินจากรูป — วัดจริงแล้วแก้ mount_offset)
+           26 ต.ค.: แขนซ้ายเปลี่ยนเป็นชุดมือซ้ายแล้ว (arm hand-side left) — รูปจริง: ฝ่ามือหันทางเดิม นิ้วโป้งอยู่ด้านนอก
+           ส่วนโมเดล (มือขวา) นิ้วโป้งอยู่ฝั่งเสา -> ใช้ mesh มือซ้าย มุมยึดเดิม -->
+      <xacro:amazinghand prefix="left_" parent="left_link_6" side="left" mount_offset="0.025" mount_yaw="${pi/2}"/>
     </xacro:if>
     <xacro:if value="${right_hand}">
-      <!-- มือซ้าย (ภาพสะท้อนของมือขวา) ยึดแบบสะท้อนกับแขนซ้าย — mount_yaw คำนวณให้ฝ่ามือสะท้อนฝ่ามือซ้ายพอดี
-           ที่ท่าพัก (ยังไม่มีรูปมือจริงบนแขนขวา — มีแล้วเทียบอีกครั้ง) -->
-      <xacro:amazinghand prefix="right_" parent="right_link_6" side="left" mount_offset="0.025"
+      <!-- ชุดมือขวาจะติดแขนขวา (ภาพสะท้อนของแขนซ้าย) — mount_yaw สะท้อนของแขนซ้าย
+           (ยังไม่มีรูปมือจริงบนแขนขวา — มีแล้วเทียบอีกครั้ง) -->
+      <xacro:amazinghand prefix="right_" parent="right_link_6" side="right" mount_offset="0.025"
                          mount_yaw="${-pi/2}"/>
     </xacro:if>
